Commit message: feat: updated xacro and launch files

File: xacro/laser.xacro (robot description, xacro)
@@ -1,5 +1,5 @@
 <?xml version="1.0" encoding="UTF-8"?>
 <robot xmlns:xacro="http://www.ros.org/wiki/xacro">
-    <xacro:macro name="standoff" params="name length radius mass">
+    <xacro:macro name="laser" params="name length radius ">
         <link name="${name}">
             <visual>
@@ -7,8 +7,9 @@
                 <geometry>
                     <!-- units in meters -->
-                    <cylinder length="${length}" radius="${radius}" />
+                    <!-- assumed solid cylinder as geometry for the sensor -->
+                    <mesh filename="package://barista_robot_description/meshes/hokuyo_urg_04lx.dae" />
                 </geometry>
-                <material name="white">
-                    <color rgba="1 1 1 0.5" />
+                <material name="yellow">
+                    <color rgba="1 1 0 1" />
                 </material>
             </visual>
@@ -23,10 +24,11 @@
                 <origin xyz="0 0 0" rpy="0 0 0" />
                 <!-- units in kilograms -->
-                <mass value="${mass}" />
+                <!-- assumed negligible mass for the sensor -->
+                <mass value="0.001" />
                 <!-- inertial tensors for solid cylinder -->
                 <inertia
-                    ixx="${mass*(3*radius*radius+length*length)/12}" ixy="0.0" ixz="0.0"
-                    iyy="${mass*(3*radius*radius+length*length)/12}" iyz="0.0"
-                    izz="${mass*(radius*radius)/2}"
+                    ixx="${0.001*(3*radius*radius+length*length)/12}" ixy="0.0" ixz="0.0"
+                    iyy="${0.001*(3*radius*radius+length*length)/12}" iyz="0.0"
+                    izz="${0.001*(radius*radius)/2}"
                 />
             </inertial>
