Commit message: fix: laser frame and added inverse parameter

File: xacro/barista_robot_model.urdf.xacro (robot description, xacro)
@@ -7,4 +7,5 @@
     <xacro:arg name="include_laser" default="true" />
     <xacro:arg name="include_joint_state" default="true" />
+    <xacro:arg name="inverse" default="false" />
     <!-- XACRO FILES -->
     <xacro:include filename="wheel.xacro" />
@@ -142,12 +143,19 @@
     <!-- GAZEBO -->
     <!-- properties for base_link -->
-    <gazebo reference="base_link">
-        <material>Gazebo/Blue </material>
-    </gazebo>
+    <xacro:if value="$(arg inverse)">
+        <gazebo reference="base_link">
+            <material>Gazebo/Red </material>
+        </gazebo>
+    </xacro:if>
+    <xacro:unless value="$(arg inverse)">
+        <gazebo reference="base_link">
+            <material>Gazebo/Blue </material>
+        </gazebo>
+    </xacro:unless>
     <!-- properties for right_wheel -->
     <gazebo reference="right_wheel">
         <mu1>1</mu1>
         <mu2>1</mu2>
-        <material>Gazebo/Red </material>
+        <material>Gazebo/White </material>
     </gazebo>
     <!-- properties for left_wheel -->
@@ -155,5 +163,5 @@
         <mu1>1</mu1>
         <mu2>1</mu2>
-        <material>Gazebo/Red </material>
+        <material>Gazebo/White </material>
     </gazebo>
     <!-- properties for front_caster -->
@@ -188,7 +196,14 @@
     </gazebo>
     <!-- properties for cup_holder -->
-    <gazebo reference="cup_holder">
-        <material>Gazebo/Blue </material>
-    </gazebo>
+    <xacro:if value="$(arg inverse)">
+        <gazebo reference="cup_holder">
+            <material>Gazebo/Red </material>
+        </gazebo>
+    </xacro:if>
+    <xacro:unless value="$(arg inverse)">
+        <gazebo reference="cup_holder">
+            <material>Gazebo/Blue </material>
+        </gazebo>
+    </xacro:unless>
     <!-- properties for base_laser -->
     <xacro:if value="$(arg include_laser)">
@@ -201,5 +216,4 @@
         <plugin filename="libgazebo_ros_diff_drive.so" name="differential_drive_controller">
             <!-- defined parameters -->
-            <robot_base_frame>base_footprint</robot_base_frame>
             <left_joint>joint_base_to_right_wheel</left_joint>
             <right_joint>joint_base_to_left_wheel</right_joint>
@@ -211,5 +225,7 @@
             <publish_odom>true</publish_odom>
             <publish_odom_tf>true</publish_odom_tf>
-            <odometry_frame>odom</odometry_frame>
+            <!-- launch parameters -->
+            <robot_base_frame>$(arg namespace)/base_footprint</robot_base_frame>
+            <odometry_frame>$(arg namespace)/odom</odometry_frame>
             <ros>
                 <namespace>$(arg namespace)</namespace>
@@ -250,6 +266,8 @@
                     <!-- defined parameters -->
                     <ros>
-                        <remapping>~/out:=$(arg namespace)/scan</remapping>
+                        <namespace>$(arg namespace)</namespace>
+                        <remapping>~/out:=scan</remapping>
                     </ros>
+                    <frame_name>$(arg namespace)/base_laser</frame_name>
                     <!-- default parameters -->
                     <output_type>sensor_msgs/LaserScan</output_type>

Commit message: fix: robot inverse property for rviz

File: xacro/barista_robot_model.urdf.xacro (robot description, xacro)
@@ -9,4 +9,5 @@
     <xacro:arg name="inverse" default="false" />
     <!-- XACRO FILES -->
+    <xacro:include filename="base.xacro" />
     <xacro:include filename="wheel.xacro" />
     <xacro:include filename="standoff.xacro" />
@@ -18,34 +19,5 @@
     </link>
     <!-- base -->
-    <link name="base_link">
-        <visual>
-            <origin xyz="0 0 0" rpy="0 0 0" />
-            <geometry>
-                <!-- units in meters -->
-                <cylinder length="0.155" radius="0.178" />
-            </geometry>
-            <material name="blue">
-                <color rgba="0 0 1 0.5" />
-            </material>
-        </visual>
-        <collision>
-            <origin xyz="0 0 0" rpy="0 0 0" />
-            <geometry>
-                <!-- units in meters -->
-                <cylinder length="0.155" radius="0.178" />
-            </geometry>
-        </collision>
-        <inertial>
-            <origin xyz="0 0 0" rpy="0 0 0" />
-            <!-- units in kilograms -->
-            <mass value="10" />
-            <!-- inertial tensors for solid cylinder -->
-            <inertia
-                ixx="0.09923" ixy="0.0" ixz="0.0"
-                iyy="0.09923" iyz="0.0"
-                izz="0.15842"
-            />
-        </inertial>
-    </link>
+    <xacro:base name="base_link" length="0.155" radius="0.178" mass="10" />
     <!-- right wheel -->
     <xacro:wheel name="right_wheel" length="0.0206" radius="0.0352" mass="1" />

File: xacro/base.xacro (robot description, xacro)
@@ -1,5 +1,5 @@
 <?xml version="1.0" encoding="UTF-8"?>
 <robot xmlns:xacro="http://www.ros.org/wiki/xacro">
-    <xacro:macro name="cup_holder_tray" params="name length radius mass">
+    <xacro:macro name="base" params="name length radius mass">
         <link name="${name}">
             <visual>

File: xacro/wheel.xacro (robot description, xacro)
@@ -9,6 +9,6 @@
                     <cylinder length="${length}" radius="${radius}" />
                 </geometry>
-                <material name="red">
-                    <color rgba="1 0 0 1" />
+                <material name="white">
+                    <color rgba="1 1 1 0.5" />
                 </material>
             </visual>
@@ -42,5 +42,5 @@
                 </geometry>
                 <material name="white">
-                    <color rgba="1 1 1 1" />
+                    <color rgba="1 1 1 0.5" />
                 </material>
             </visual>
